File: FourthAxis/Handwheel.kicad_sch (KiCad schematic)
At the start: 0 parts

Commit message: started handwheel
Parts:
- added R11, R12, R5, R6: 1k, symbol Device:R_US
- added U5: LMV393, symbol Comparator:LMV393
Connections:
- new net: R5.2, U5.1
- new net: R11.2, R12.1, U5.2 (-), U5.6 (-)
- new net: R6.2, U5.7
- new net 3V3: R11.1, R5.1, R6.1, U5.8 (V+)
- new net ENC_A_5V: U5.3 (+)
- new net ENC_B_5V: U5.5 (+)
- new net GND: R12.2, U5.4 (V-)

Commit message: schem additions
Parts:
- removed R5, R6: 1k, symbol Device:R_US
- removed U5: LMV393, symbol Comparator:LMV393
- added U6, U7: SN74LVC1T45DBV, Package_TO_SOT_SMD:SOT-23-6, symbol Logic_LevelTranslator:SN74LVC1T45DBV
- R11, R12: value 1k -> 10k
Connections:
- net 3V3: now also U6.6 (VCCB), U7.6 (VCCB); no longer R11.1
- net GND: now also U6.2 (GND), U7.2 (GND); no longer R12.2
- net at R11.2: now also U6.5 (DIR); no longer R12.1
- new net: R12.2, U7.5 (DIR)
- new net 5V: R11.1, R12.1, U6.1 (VCCA), U7.1 (VCCA)
- new net ENC_A_IN: U6.3 (A)
- new net ENC_B_IN: U7.3 (A)
- new net HAND_DIR: U7.4 (B)
- new net HAND_INT: U6.4 (B)

Commit message: name and layout
Parts:
- R11, R12: footprint (none) -> Resistor_SMD:R_0603_1608Metric
Changed lines of the file:
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@@
 			)
 		)
-		(property "Footprint" ""
+		(property "Footprint" "Resistor_SMD:R_0603_1608Metric"
 			(at 68.834 97.536 90)
 			(hide yes)
@@
 			)
 		)
-		(property "Footprint" ""
+		(property "Footprint" "Resistor_SMD:R_0603_1608Metric"
 			(at 67.564 59.436 90)
 			(hide yes)

Commit message: Nick end of wed
Other:
- moved on the sheet: R11, R12, U6, U7

Commit message: digikey PN and footprints
Parts:
- R10: renamed from R12; digikey (none) -> 311-10.0KHRCT-ND
- R9: renamed from R11; digikey (none) -> 311-10.0KHRCT-ND
- U3: renamed from U6; digikey (none) -> 296-16843-1-ND
- U4: renamed from U7; digikey (none) -> 296-16843-1-ND
Changed lines of the file:
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@@
 		(dnp no)
 		(fields_autoplaced yes)
-		(property "Reference" "U7"
+		(property "Reference" "U4"
 			(at 119.38 71.0498 0)
 			(show_name no)
@@
 		)
 		(property "Digikey" "74LVC1T45W6-7DICT-ND"
+			(at 101.6 77.47 0)
+			(hide yes)
+			(show_name no)
+			(do_not_autoplace no)
+			(effects
+				(font
+					(size 1.27 1.27)
+				)
+			)
+		)
+		(property "digikey" "296-16843-1-ND"
 			(at 101.6 77.47 0)
 			(hide yes)
@@
 			(project "FourthAxis"
 				(path "/32b0d774-33bf-42ba-9d9e-f33866433972/0e7e279c-42fe-4d5f-ab1e-1661f1173f00"
-					(reference "U7")
+					(reference "U4")
 					(unit 1)
 				)
@@
 		(in_pos_files yes)
 		(dnp no)
-		(property "Reference" "R12"
+		(property "Reference" "R10"
 			(at 83.82 88.9 90)
 			(show_name no)
@@
 		(property "Description" "Resistor, US symbol"
 			(at 83.82 82.55 0)
+			(hide yes)
+			(show_name no)
+			(do_not_autoplace no)
+			(effects
+				(font
+					(size 1.27 1.27)
+				)
+			)
+		)
+		(property "digikey" "311-10.0KHRCT-ND"
+			(at 83.82 82.55 90)
 			(hide yes)
 			(show_name no)
@@
 			(project "FourthAxis"
 				(path "/32b0d774-33bf-42ba-9d9e-f33866433972/0e7e279c-42fe-4d5f-ab1e-1661f1173f00"
-					(reference "R12")
+					(reference "R10")
 					(unit 1)
 				)
@@
 		(in_pos_files yes)
 		(dnp no)
-		(property "Reference" "R11"
+		(property "Reference" "R9"
 			(at 83.82 50.8 90)
 			(show_name no)
@@
 		(property "Description" "Resistor, US symbol"
 			(at 83.82 44.45 0)
+			(hide yes)
+			(show_name no)
+			(do_not_autoplace no)
+			(effects
+				(font
+					(size 1.27 1.27)
+				)
+			)
+		)
+		(property "digikey" "311-10.0KHRCT-ND"
+			(at 83.82 44.45 90)
 			(hide yes)
 			(show_name no)
@@
 			(project "FourthAxis"
 				(path "/32b0d774-33bf-42ba-9d9e-f33866433972/0e7e279c-42fe-4d5f-ab1e-1661f1173f00"
-					(reference "R11")
+					(reference "R9")
 					(unit 1)
 				)
@@
 		(dnp no)
 		(fields_autoplaced yes)
-		(property "Reference" "U6"
+		(property "Reference" "U3"
 			(at 119.38 32.9498 0)
 			(show_name no)
@@
 		)
 		(property "Digikey" "74LVC1T45W6-7DICT-ND"
+			(at 101.6 39.37 0)
+			(hide yes)
+			(show_name no)
+			(do_not_autoplace no)
+			(effects
+				(font
+					(size 1.27 1.27)
+				)
+			)
+		)
+		(property "digikey" "296-16843-1-ND"
 			(at 101.6 39.37 0)
 			(hide yes)
@@
 			(project "FourthAxis"
 				(path "/32b0d774-33bf-42ba-9d9e-f33866433972/0e7e279c-42fe-4d5f-ab1e-1661f1173f00"
-					(reference "U6")
+					(reference "U3")
 					(unit 1)
 				)
