File: FourthAxis/PD.kicad_sch (KiCad schematic)
At the start: 2 parts, among them U3 XL1509-5.0, U4 XL1509-3.3

Commit message: Shaun work
Parts:
- added C1, C4: 470u, symbol Device:C_US
- added C2, C5: 1u, symbol Device:C
- added C3, C6: 330u, symbol Device:C_US
- added D27, D28: 1N5821, Diode_THT:D_DO-201AD_P15.24mm_Horizontal, symbol Diode:1N5821
- added L1: 68u, symbol Device:L
- added L2: 47u, symbol Device:L
- added R16, R17: 10k, symbol Device:R_US
Connections:
- net 12V: now reaches U3.1 (VIN)
- net 12V: now also U4.1 (VIN), C1.1, C2.1, C4.1, C5.1
- net at U3.2 (OUT): now also D27.1 (K), L1.1
- net 5V: now reaches U3.3 (FB)
- net 5V: now also C3.1, L1.2
- net at U3.4 (~{EN}): now also R16.1
- net GND: now reaches U3.5 (GND), U3.6 (GND), U3.7 (GND), U3.8 (GND)
- net GND: now also U4.5 (GND), U4.6 (GND), U4.7 (GND), U4.8 (GND), C1.2, C2.2, C3.2, C4.2, C5.2, C6.2, D27.2 (A), D28.2 (A), R16.2, R17.2
- net at U4.2 (OUT): now also D28.1 (K), L2.1
- net 3V3: now reaches U4.3 (FB)
- net 3V3: now also C6.1, L2.2
- net at U4.4 (~{EN}): now also R17.1
Other:
- moved on the sheet: U3, U4

Commit message: shaun today
Parts:
- C1, C4: footprint (none) -> Capacitor_SMD:CP_Elec_16x17.5; digikey (none) -> 493-UUG1H471MNJ6MSCT-ND
- C2, C5: footprint (none) -> Capacitor_SMD:C_0805_2012Metric; digikey (none) -> 2679-AGC0805X7R500-105KNETR-ND
- C3, C6: footprint (none) -> Capacitor_SMD:CP_Elec_6.3x7.7; digikey (none) -> 493-2157-1-ND
- L1: footprint (none) -> Inductor_SMD:L_12x12mm_H6mm
- L2: footprint (none) -> Inductor_SMD:L_12x12mm_H6mm; digikey (none) -> 399-MPXV1D1250L470CT-ND
- R16, R17: footprint (none) -> Resistor_SMD:R_0402_1005Metric; digikey (none) -> 311-10.0KLRCT-ND
Connections:
- net 12V renamed 36V
Changed lines of the file:
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@@
 		)
 	)
-	(hierarchical_label "12V"
+	(hierarchical_label "36V"
 		(shape input)
 		(at 151.13 63.5 180)
@@
 		)
 	)
-	(hierarchical_label "12V"
+	(hierarchical_label "36V"
 		(shape input)
 		(at 38.1 63.5 180)
@@
 			)
 		)
-		(property "Footprint" ""
+		(property "Footprint" "Resistor_SMD:R_0402_1005Metric"
 			(at 185.166 76.454 90)
 			(hide yes)
@@
 			)
 		)
-		(property "Datasheet" ""
+		(property "Datasheet" "https://www.digikey.com/en/products/detail/yageo/RC0402FR-0710KL/726523"
 			(at 184.15 76.2 0)
 			(hide yes)
@@
 		)
 		(property "Description" "Resistor, US symbol"
+			(at 184.15 76.2 0)
+			(hide yes)
+			(show_name no)
+			(do_not_autoplace no)
+			(effects
+				(font
+					(size 1.27 1.27)
+				)
+			)
+		)
+		(property "digikey" "311-10.0KLRCT-ND"
 			(at 184.15 76.2 0)
 			(hide yes)
@@
 			)
 		)
-		(property "Footprint" ""
+		(property "Footprint" "Inductor_SMD:L_12x12mm_H6mm"
 			(at 227.33 63.5 0)
 			(hide yes)
@@
 			)
 		)
-		(property "Datasheet" ""
+		(property "Datasheet" "https://www.digikey.com/en/products/detail/kemet/MPXV1D1250L470/11314587?s=N4IgTCBcDaILIAUAaA1AjAETWArABgBkAWAdjxAF0BfIA"
 			(at 227.33 63.5 0)
 			(hide yes)
@@
 		(property "Description" "Inductor"
 			(at 227.33 63.5 0)
+			(hide yes)
+			(show_name no)
+			(do_not_autoplace no)
+			(effects
+				(font
+					(size 1.27 1.27)
+				)
+			)
+		)
+		(property "digikey" "399-MPXV1D1250L470CT-ND"
+			(at 227.33 63.5 90)
 			(hide yes)
 			(show_name no)
@@
 			)
 		)
-		(property "Footprint" ""
+		(property "Footprint" "Capacitor_SMD:CP_Elec_6.3x7.7"
 			(at 237.49 76.2 0)
 			(hide yes)
@@
 			)
 		)
-		(property "Datasheet" ""
+		(property "Datasheet" "https://www.digikey.com/en/products/detail/nichicon/UWT0J331MCL1GS/589898"
 			(at 237.49 76.2 0)
 			(hide yes)
@@
 		)
 		(property "Description" "capacitor, US symbol"
+			(at 237.49 76.2 0)
+			(hide yes)
+			(show_name no)
+			(do_not_autoplace no)
+			(effects
+				(font
+					(size 1.27 1.27)
+				)
+			)
+		)
+		(property "digikey" "493-2157-1-ND"
 			(at 237.49 76.2 0)
 			(hide yes)
@@
 			)
 		)
-		(property "Footprint" ""
+		(property "Footprint" "Capacitor_SMD:CP_Elec_16x17.5"
 			(at 45.72 73.66 0)
 			(hide yes)
@@
 			)
 		)
-		(property "Datasheet" ""
+		(property "Datasheet" "https://www.digikey.com/en/products/detail/nichicon/UUG1H471MNJ6MS/3768773"
 			(at 45.72 73.66 0)
 			(hide yes)
@@
 		)
 		(property "Description" "capacitor, US symbol"
+			(at 45.72 73.66 0)
+			(hide yes)
+			(show_name no)
+			(do_not_autoplace no)
+			(effects
+				(font
+					(size 1.27 1.27)
+				)
+			)
+		)
+		(property "digikey" "493-UUG1H471MNJ6MSCT-ND"
 			(at 45.72 73.66 0)
 			(hide yes)
@@
 			)
 		)
-		(property "Footprint" ""
+		(property "Footprint" "Inductor_SMD:L_12x12mm_H6mm"
 			(at 114.3 63.5 0)
 			(hide yes)
@@
 			)
 		)
-		(property "Datasheet" ""
+		(property "Datasheet" "https://www.digikey.com/en/products/detail/kemet/MPXV1D1250L680/11314689?s=N4IgTCBcDaIMwE4EFoCyAFAGgNQIwBFcwBWABgBkA2ADlIGEAVZAOXxAF0BfIA"
 			(at 114.3 63.5 0)
 			(hide yes)
@@
 			)
 		)
-		(property "Footprint" ""
+		(property "Footprint" "Capacitor_SMD:CP_Elec_6.3x7.7"
 			(at 124.46 76.2 0)
 			(hide yes)
-			(show_name no)
-			(do_not_autoplace no)
-			(effects
-				(font
-					(size 1.27 1.27)
-				)
-			)
-		)
-		(property "Datasheet" ""
+			(show_name yes)
+			(do_not_autoplace no)
+			(effects
+				(font
+					(size 1.27 1.27)
+				)
+			)
+		)
+		(property "Datasheet" "https://www.digikey.com/en/products/detail/nichicon/UWT0J331MCL1GS/589898"
 			(at 124.46 76.2 0)
 			(hide yes)
@@
 		)
 		(property "Description" "capacitor, US symbol"
+			(at 124.46 76.2 0)
+			(hide yes)
+			(show_name no)
+			(do_not_autoplace no)
+			(effects
+				(font
+					(size 1.27 1.27)
+				)
+			)
+		)
+		(property "digikey" "493-2157-1-ND"
 			(at 124.46 76.2 0)
 			(hide yes)
@@
 			)
 		)
-		(property "Footprint" ""
+		(property "Footprint" "Capacitor_SMD:CP_Elec_16x17.5"
 			(at 158.75 73.66 0)
 			(hide yes)
@@
 			)
 		)
-		(property "Datasheet" ""
+		(property "Datasheet" "https://www.digikey.com/en/products/detail/nichicon/UUG1H471MNJ6MS/3768773"
 			(at 158.75 73.66 0)
 			(hide yes)
@@
 		)
 		(property "Description" "capacitor, US symbol"
+			(at 158.75 73.66 0)
+			(hide yes)
+			(show_name no)
+			(do_not_autoplace no)
+			(effects
+				(font
+					(size 1.27 1.27)
+				)
+			)
+		)
+		(property "digikey" "493-UUG1H471MNJ6MSCT-ND"
 			(at 158.75 73.66 0)
 			(hide yes)
@@
 			)
 		)
-		(property "Footprint" ""
+		(property "Footprint" "Capacitor_SMD:C_0805_2012Metric"
 			(at 173.6852 77.47 0)
 			(hide yes)
@@
 			)
 		)
-		(property "Datasheet" ""
+		(property "Datasheet" "https://www.digikey.com/en/products/detail/venkel/AGC0805X7R500-105KNE/20485164?s=N4IgTCBcDa4GwHYCcBaAggcQMIAYAcOArABoIBKhOOKAjEQNIByAogCpkqMAiIAugL5A"
 			(at 172.72 73.66 0)
 			(hide yes)
@@
 		)
 		(property "Description" "Unpolarized capacitor"
+			(at 172.72 73.66 0)
+			(hide yes)
+			(show_name no)
+			(do_not_autoplace no)
+			(effects
+				(font
+					(size 1.27 1.27)
+				)
+			)
+		)
+		(property "digikey" "2679-AGC0805X7R500-105KNETR-ND"
 			(at 172.72 73.66 0)
 			(hide yes)
@@
 			)
 		)
-		(property "Footprint" ""
+		(property "Footprint" "Resistor_SMD:R_0402_1005Metric"
 			(at 72.136 76.454 90)
 			(hide yes)
@@
 			)
 		)
-		(property "Datasheet" ""
+		(property "Datasheet" "https://www.digikey.com/en/products/detail/yageo/RC0402FR-0710KL/726523"
 			(at 71.12 76.2 0)
 			(hide yes)
@@
 		)
 		(property "Description" "Resistor, US symbol"
+			(at 71.12 76.2 0)
+			(hide yes)
+			(show_name no)
+			(do_not_autoplace no)
+			(effects
+				(font
+					(size 1.27 1.27)
+				)
+			)
+		)
+		(property "digikey" "311-10.0KLRCT-ND"
 			(at 71.12 76.2 0)
 			(hide yes)
@@
 			)
 		)
-		(property "Footprint" ""
+		(property "Footprint" "Capacitor_SMD:C_0805_2012Metric"
 			(at 60.6552 77.47 0)
 			(hide yes)
@@
 			)
 		)
-		(property "Datasheet" ""
+		(property "Datasheet" "https://www.digikey.com/en/products/detail/venkel/AGC0805X7R500-105KNE/20485164?s=N4IgTCBcDa4GwHYCcBaAggcQMIAYAcOArABoIBKhOOKAjEQNIByAogCpkqMAiIAugL5A"
 			(at 59.69 73.66 0)
 			(hide yes)
@@
 			(at 59.69 73.66 0)
 			(hide yes)
+			(show_name no)
+			(do_not_autoplace no)
+			(effects
+				(font
+					(size 1.27 1.27)
+				)
+			)
+		)
+		(property "digikey" "2679-AGC0805X7R500-105KNETR-ND"
+			(at 59.69 73.66 0)
+			(hide yes)

Commit message: Encoder input added?
Changed lines of the file:
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@@
 	)
 	(hierarchical_label "5V"
-		(shape input)
+		(shape output)
 		(at 134.62 68.58 0)
 		(effects
@@
 	)
 	(hierarchical_label "3V3"
-		(shape input)
+		(shape output)
 		(at 247.65 68.58 0)
 		(effects

Commit message: digikey PN and footprints
Parts:
- C1, C4: footprint Capacitor_SMD:CP_Elec_16x17.5 -> Capacitor_THT:C_Radial_D10.0mm_H20.0mm_P5.00mm; digikey 493-UUG1H471MNJ6MSCT-ND -> P5185-ND
- C2, C5: footprint Capacitor_SMD:C_0805_2012Metric -> Capacitor_SMD:C_0603_1608Metric; digikey 2679-AGC0805X7R500-105KNETR-ND -> 1276-1184-1-ND
- D27, D28: footprint Diode_THT:D_DO-201AD_P15.24mm_Horizontal -> Diode_SMD:D_SOD-123; digikey (none) -> 641-1458-1-ND
- R11: renamed from R16; footprint Resistor_SMD:R_0402_1005Metric -> Resistor_SMD:R_0603_1608Metric; digikey 311-10.0KLRCT-ND -> 311-10.0KHRCT-ND
- R12: renamed from R17; footprint Resistor_SMD:R_0402_1005Metric -> Resistor_SMD:R_0603_1608Metric; digikey 311-10.0KLRCT-ND -> 311-10.0KHRCT-ND
- U5: renamed from U3; digikey (none) -> 4518-XL1509-5.0CT-ND
- U6: renamed from U4; digikey (none) -> 4518-XL1509-3.3CT-ND
Changed lines of the file:
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@@
 		(dnp no)
 		(fields_autoplaced yes)
-		(property "Reference" "R17"
+		(property "Reference" "R12"
 			(at 186.69 74.9299 0)
 			(show_name no)
@@
 			)
 		)
-		(property "Footprint" "Resistor_SMD:R_0402_1005Metric"
+		(property "Footprint" "Resistor_SMD:R_0603_1608Metric"
 			(at 185.166 76.454 90)
 			(hide yes)
@@
 			)
 		)
-		(property "digikey" "311-10.0KLRCT-ND"
+		(property "digikey" "311-10.0KHRCT-ND"
 			(at 184.15 76.2 0)
 			(hide yes)
@@
 			(project "FourthAxis"
 				(path "/32b0d774-33bf-42ba-9d9e-f33866433972/39636035-34df-404d-b7c8-3e3bf34934f2"
-					(reference "R17")
+					(reference "R12")
 					(unit 1)
 				)
@@
 			)
 		)
-		(property "Footprint" "Diode_THT:D_DO-201AD_P15.24mm_Horizontal"
+		(property "Footprint" "Diode_SMD:D_SOD-123"
 			(at 213.995 76.2 0)
 			(hide yes)
@@
 		(property "Description" "30V 3A Schottky Barrier Rectifier Diode, DO-201AD"
 			(at 218.44 76.2 0)
+			(hide yes)
+			(show_name no)
+			(do_not_autoplace no)
+			(effects
+				(font
+					(size 1.27 1.27)
+				)
+			)
+		)
+		(property "digikey" "641-1458-1-ND"
+			(at 218.44 76.2 90)
 			(hide yes)
 			(show_name no)
@@
 			)
 		)
-		(property "Footprint" "Capacitor_SMD:CP_Elec_16x17.5"
+		(property "Footprint" "Capacitor_THT:C_Radial_D10.0mm_H20.0mm_P5.00mm"
 			(at 45.72 73.66 0)
 			(hide yes)
@@
 			)
 		)
-		(property "digikey" "493-UUG1H471MNJ6MSCT-ND"
+		(property "digikey" "P5185-ND"
 			(at 45.72 73.66 0)
 			(hide yes)
@@
 			)
 		)
-		(property "Footprint" "Capacitor_SMD:CP_Elec_16x17.5"
+		(property "Footprint" "Capacitor_THT:C_Radial_D10.0mm_H20.0mm_P5.00mm"
 			(at 158.75 73.66 0)
 			(hide yes)
@@
 			)
 		)
-		(property "digikey" "493-UUG1H471MNJ6MSCT-ND"
+		(property "digikey" "P5185-ND"
 			(at 158.75 73.66 0)
 			(hide yes)
@@
 			)
 		)
-		(property "Footprint" "Diode_THT:D_DO-201AD_P15.24mm_Horizontal"
+		(property "Footprint" "Diode_SMD:D_SOD-123"
 			(at 100.965 76.2 0)
 			(hide yes)
@@
 		(property "Description" "30V 3A Schottky Barrier Rectifier Diode, DO-201AD"
 			(at 105.41 76.2 0)
+			(hide yes)
+			(show_name no)
+			(do_not_autoplace no)
+			(effects
+				(font
+					(size 1.27 1.27)
+				)
+			)
+		)
+		(property "digikey" "641-1458-1-ND"
+			(at 105.41 76.2 90)
 			(hide yes)
 			(show_name no)
@@
 			)
 		)
-		(property "Footprint" "Capacitor_SMD:C_0805_2012Metric"
+		(property "Footprint" "Capacitor_SMD:C_0603_1608Metric"
 			(at 173.6852 77.47 0)
 			(hide yes)
@@
 			)
 		)
-		(property "digikey" "2679-AGC0805X7R500-105KNETR-ND"
+		(property "digikey" "1276-1184-1-ND"
 			(at 172.72 73.66 0)
 			(hide yes)
@@
 		(dnp no)
 		(fields_autoplaced yes)
-		(property "Reference" "U3"
+		(property "Reference" "U5"
 			(at 88.9 55.88 0)
 			(show_name no)
@@
 			)
 		)
+		(property "digikey" "4518-XL1509-5.0CT-ND"
+			(at 88.9 66.04 0)
+			(hide yes)
+			(show_name no)
+			(do_not_autoplace no)
+			(effects
+				(font
+					(size 1.27 1.27)
+				)
+			)
+		)
 		(pin "6"
 		)
@@
 			(project "FourthAxis"
 				(path "/32b0d774-33bf-42ba-9d9e-f33866433972/39636035-34df-404d-b7c8-3e3bf34934f2"
-					(reference "U3")
+					(reference "U5")
 					(unit 1)
 				)
@@
 		(dnp no)
 		(fields_autoplaced yes)
-		(property "Reference" "R16"
+		(property "Reference" "R11"
 			(at 73.66 74.9299 0)
 			(show_name no)
@@
 			)
 		)
-		(property "Footprint" "Resistor_SMD:R_0402_1005Metric"
+		(property "Footprint" "Resistor_SMD:R_0603_1608Metric"
 			(at 72.136 76.454 90)
 			(hide yes)
@@
 			)
 		)
-		(property "digikey" "311-10.0KLRCT-ND"
+		(property "digikey" "311-10.0KHRCT-ND"
 			(at 71.12 76.2 0)
 			(hide yes)
@@
 			(project "FourthAxis"
 				(path "/32b0d774-33bf-42ba-9d9e-f33866433972/39636035-34df-404d-b7c8-3e3bf34934f2"
-					(reference "R16")
+					(reference "R11")
 					(unit 1)
 				)
@@
 			)
 		)
-		(property "Footprint" "Capacitor_SMD:C_0805_2012Metric"
+		(property "Footprint" "Capacitor_SMD:C_0603_1608Metric"
 			(at 60.6552 77.47 0)
 			(hide yes)
@@
 			)
 		)
-		(property "digikey" "2679-AGC0805X7R500-105KNETR-ND"
+		(property "digikey" "1276-1184-1-ND"
 			(at 59.69 73.66 0)
 			(hide yes)
@@
 		(dnp no)
 		(fields_autoplaced yes)
-		(property "Reference" "U4"
+		(property "Reference" "U6"
 			(at 201.93 55.88 0)
 			(show_name no)
@@
 			)
 		)
+		(property "digikey" "4518-XL1509-3.3CT-ND"
+			(at 201.93 66.04 0)
+			(hide yes)
+			(show_name no)
+			(do_not_autoplace no)
+			(effects
+				(font
+					(size 1.27 1.27)
+				)
+			)
+		)
 		(pin "2"
 		)
@@
 			(project "FourthAxis"
 				(path "/32b0d774-33bf-42ba-9d9e-f33866433972/39636035-34df-404d-b7c8-3e3bf34934f2"
-					(reference "U4")
-					(unit 1)
-				)
+					(reference "U6")
+					(unit 1)
+				)
