File: FourthAxis/PD.kicad_sch (KiCad schematic)
At the start: 17 parts, among them U5 XL1509-5.0, U6 XL1509-3.3

Commit message: boards ordered
Parts:
- C28, C29: digikey 1276-1184-1-ND -> 1292-0603X106M100CT-ND
Changed lines of the file:
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@@
 			)
 		)
-		(property "digikey" "1276-1184-1-ND"
+		(property "digikey" "1292-0603X106M100CT-ND"
 			(at 64.77 31.75 0)
 			(hide yes)
@@
 			)
 		)
-		(property "digikey" "1276-1184-1-ND"
+		(property "digikey" "1292-0603X106M100CT-ND"
 			(at 54.61 31.75 0)
 			(hide yes)
