File: FourthAxis/FourthAxis.kicad_sch (KiCad schematic)
At the start: 1 part, among them U1 ESP32-WROOM-32

Commit message: Progress save
Other:
- added sheet KeyPad (KeyPad.kicad_sch)
Changed lines of the file:
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@@
+		)
+	)
+	(sheet
+		(at 214.63 87.63)
+		(size 34.29 21.59)
+		(exclude_from_sim no)
+		(in_bom yes)
+		(on_board yes)
+		(dnp no)
+		(fields_autoplaced yes)
+		(stroke
+			(width 0.1524)
+			(type solid)
+		)
+		(fill
+			(color 0 0 0 0.0000)
+		)
+		(property "Sheetname" "KeyPad"
+			(at 214.63 86.9184 0)
+			(effects
+				(font
+					(size 1.27 1.27)
+				)
+				(justify left bottom)
+			)
+		)
+		(property "Sheetfile" "KeyPad.kicad_sch"
+			(at 214.63 109.8046 0)
+			(effects
+				(font
+					(size 1.27 1.27)
+				)
+				(justify left top)
+			)
+		)
+		(instances
+			(project "FourthAxis"
+				(path "/32b0d774-33bf-42ba-9d9e-f33866433972"
+					(page "2")
+				)
+			)
 		)
 	)

Commit message: Added handwheel sheet
Other:
- added sheet HandWheel (Handwheel.kicad_sch)
Changed lines of the file:
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@@
 	)
 	(sheet
-		(at 214.63 87.63)
+		(at 180.34 80.01)
+		(size 33.02 19.05)
+		(exclude_from_sim no)
+		(in_bom yes)
+		(on_board yes)
+		(dnp no)
+		(fields_autoplaced yes)
+		(stroke
+			(width 0.1524)
+			(type solid)
+		)
+		(fill
+			(color 0 0 0 0.0000)
+		)
+		(property "Sheetname" "HandWheel"
+			(at 180.34 79.2984 0)
+			(effects
+				(font
+					(size 1.27 1.27)
+				)
+				(justify left bottom)
+			)
+		)
+		(property "Sheetfile" "Handwheel.kicad_sch"
+			(at 180.34 99.6446 0)
+			(effects
+				(font
+					(size 1.27 1.27)
+				)
+				(justify left top)
+			)
+		)
+		(instances
+			(project "FourthAxis"
+				(path "/32b0d774-33bf-42ba-9d9e-f33866433972"
+					(page "3")
+				)
+			)
+		)
+	)
+	(sheet
+		(at 177.8 121.92)
 		(size 34.29 21.59)
 		(exclude_from_sim no)
@@
 		)
 		(property "Sheetname" "KeyPad"
-			(at 214.63 86.9184 0)
+			(at 177.8 121.2084 0)
 			(effects
 				(font
@@
 		)
 		(property "Sheetfile" "KeyPad.kicad_sch"
-			(at 214.63 109.8046 0)
+			(at 177.8 144.0946 0)
 			(effects
 				(font

Commit message: Added PD sheet
Other:
- added sheet Power Distribution (PD.kicad_sch)
Changed lines of the file:
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@@
+	)
+	(sheet
+		(at 39.37 71.12)
+		(size 35.56 25.4)
+		(exclude_from_sim no)
+		(in_bom yes)
+		(on_board yes)
+		(dnp no)
+		(fields_autoplaced yes)
+		(stroke
+			(width 0.1524)
+			(type solid)
+		)
+		(fill
+			(color 0 0 0 0)
+		)
+		(property "Sheetname" "Power Distribution"
+			(at 39.37 70.4084 0)
+			(show_name no)
+			(do_not_autoplace no)
+			(effects
+				(font
+					(size 1.27 1.27)
+				)
+				(justify left bottom)
+			)
+		)
+		(property "Sheetfile" "PD.kicad_sch"
+			(at 39.37 97.1046 0)
+			(show_name no)
+			(do_not_autoplace no)
+			(effects
+				(font
+					(size 1.27 1.27)
+				)
+				(justify left top)
+			)
+		)
+		(instances
+			(project "FourthAxis"
+				(path "/32b0d774-33bf-42ba-9d9e-f33866433972"
+					(page "4")
+				)
+			)
+		)
 	)
 	(sheet

Commit message: Keypad schem work
Connections:
- net KEY_5: no longer names the net of U1.31 (IO19)
Other:
- sheet KeyPad ports: added 3V3, KEY_1, KEY_2, KEY_3, KEY_4, KEY_A, KEY_B, KEY_C; removed none

Commit message: started handwheel
Connections:
- net KEY_6 is gone; now on net KNOB_1: U1.37 (IO23)
- net KEY_7 is gone; now on net KNOB_2: U1.10 (IO25)
- net HAND_INT: now also U1.26 (IO4); no longer U1.34 (RXD0/IO3)
- net KNOB_1: no longer U1.24 (IO2)
- net KNOB_2: no longer U1.26 (IO4)
- no-connect marks 9 -> 10

Commit message: schem additions
Parts:
- added J1: Conn_01x04_Socket, symbol Connector:Conn_01x04_Socket
Connections:
- net GND: now also J1.1 (Pin_1)
- new net 5V: J1.2 (Pin_2)
- new net HAND_INC_A: J1.4 (Pin_4)
- new net HAND_INC_B: J1.3 (Pin_3)
- no-connect marks 10 -> 12
Other:
- added sheet Knobs (Knobs.kicad_sch)
- sheet HandWheel ports: added 3V3, 5V, ENC_A_IN, ENC_B_IN, HAND_DIR, HAND_INT; removed none

Commit message: Shaun work
Other:
- sheet Power Distribution ports: added 12V, 3V3, 5V; removed none
Changed lines of the file:
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@@
+	(wire
+		(pts
+			(xy 74.93 83.82) (xy 83.82 83.82)
+		)
+		(stroke
+			(width 0)
+			(type default)
+		)
+	)
 	(wire
 		(pts
@@
 	(wire
 		(pts
+			(xy 33.02 77.47) (xy 39.37 77.47)
+		)
+		(stroke
+			(width 0)
+			(type default)
+		)
+	)
+	(wire
+		(pts
 			(xy 199.39 101.6) (xy 204.47 101.6)
 		)
@@
 	(wire
 		(pts
+			(xy 74.93 77.47) (xy 83.82 77.47)
+		)
+		(stroke
+			(width 0)
+			(type default)
+		)
+	)
+	(wire
+		(pts
 			(xy 199.39 64.77) (xy 204.47 64.77)
 		)
@@
 		)
 	)
+	(global_label "3V3"
+		(shape input)
+		(at 83.82 83.82 0)
+		(fields_autoplaced yes)
+		(effects
+			(font
+				(size 1.27 1.27)
+			)
+			(justify left)
+		)
+		(property "Intersheetrefs" "${INTERSHEET_REFS}"
+			(at 90.3128 83.82 0)
+			(hide yes)
+			(show_name no)
+			(do_not_autoplace no)
+			(effects
+				(font
+					(size 1.27 1.27)
+				)
+				(justify left)
+			)
+		)
+	)
 	(global_label "KEY_B"
 		(shape input)
@@
 		)
 	)
+	(global_label "5V"
+		(shape input)
+		(at 83.82 77.47 0)
+		(fields_autoplaced yes)
+		(effects
+			(font
+				(size 1.27 1.27)
+			)
+			(justify left)
+		)
+		(property "Intersheetrefs" "${INTERSHEET_REFS}"
+			(at 89.1033 77.47 0)
+			(hide yes)
+			(show_name no)
+			(do_not_autoplace no)
+			(effects
+				(font
+					(size 1.27 1.27)
+				)
+				(justify left)
+			)
+		)
+	)
 	(global_label "KEY_4"
 		(shape input)
@@
 		(property "Intersheetrefs" "${INTERSHEET_REFS}"
 			(at 190.7201 106.68 0)
+			(hide yes)
+			(show_name no)
+			(do_not_autoplace no)
+			(effects
+				(font
+					(size 1.27 1.27)
+				)
+				(justify right)
+			)
+		)
+	)
+	(global_label "12V"
+		(shape input)
+		(at 33.02 77.47 180)
+		(fields_autoplaced yes)
+		(effects
+			(font
+				(size 1.27 1.27)
+			)
+			(justify right)
+		)
+		(property "Intersheetrefs" "${INTERSHEET_REFS}"
+			(at 26.5272 77.47 0)
 			(hide yes)
 			(show_name no)
@@
 			)
 		)
+		(pin "12V" input
+			(at 39.37 77.47 180)
+			(effects
+				(font
+					(size 1.27 1.27)
+				)
+				(justify left)
+			)
+		)
+		(pin "5V" input
+			(at 74.93 77.47 0)
+			(effects
+				(font
+					(size 1.27 1.27)
+				)
+				(justify right)
+			)
+		)
+		(pin "3V3" input
+			(at 74.93 83.82 0)
+			(effects
+				(font
+					(size 1.27 1.27)
+				)
+				(justify right)
+			)
+		)
