File: FourthAxis/FourthAxis.kicad_sch (KiCad schematic)
At the start: 3 parts, among them J1 Conn_01x04_Socket, J2 Conn_01x08_Socket, U1 ESP32-WROOM-32

Commit message: shaunconnectors
Parts:
- added J3: DRIVER_CONN, Connector_PinHeader_2.54mm:PinHeader_1x05_P2.54mm_Vertical, symbol Connector:Conn_01x05_Socket
- added J4: 36V POWER IN, Connector_PinHeader_2.54mm:PinHeader_1x02_P2.54mm_Vertical, symbol Connector:Conn_01x02_Pin
- J1: value Conn_01x04_Socket -> HW_CONN; footprint (none) -> Connector_PinHeader_2.54mm:PinHeader_1x04_P2.54mm_Vertical
- J2: value Conn_01x08_Socket -> ENC_CONN; footprint (none) -> Connector_PinHeader_2.54mm:PinHeader_1x08_P2.54mm_Vertical
Connections:
- net GND: now also J3.5 (Pin_5), J4.2 (Pin_2)
- net MotorDriveOut/ALR_IN: now also J3.4 (Pin_4)
- net MotorDriveOut/DIR_OUT: now also J3.2 (Pin_2)
- net MotorDriveOut/EN_OUT: now also J3.3 (Pin_3)
- net MotorDriveOut/STP_OUT: now also J3.1 (Pin_1)
- new net Power Distribution/36V: J4.1 (Pin_1)

Commit message: digikey PN and footprints
Parts:
- U1: Digikey Part Number (none) -> 1965-ESP32-WROOM-32E-N4CT-ND; digikey (none) -> 1965-ESP32-WROOM-32E-N4CT-ND
- renumbered J4 to J1, J3 to J2, J2 to J3, J1 to J4
Other:
- moved on the sheet: J1, J3

Commit message: Layout work
Parts:
- added R27: 10k, Resistor_SMD:R_0603_1608Metric, symbol Device:R_US
- added SW29: BOOT, Button_Switch_SMD:SW_Push_1P1T_NO_CK_KMR2, symbol Switch:SW_Push
- added SW30: RESET, Button_Switch_SMD:SW_Push_1P1T_NO_CK_KMR2, symbol Switch:SW_Push
- J1: footprint Connector_PinHeader_2.54mm:PinHeader_1x02_P2.54mm_Vertical -> Connector_PinHeader_2.54mm:PinHeader_1x02_P2.54mm_Horizontal
- J2: footprint Connector_PinHeader_2.54mm:PinHeader_1x05_P2.54mm_Vertical -> Connector_PinHeader_2.54mm:PinHeader_1x05_P2.54mm_Horizontal
- J3: footprint Connector_PinHeader_2.54mm:PinHeader_1x08_P2.54mm_Vertical -> Connector_PinHeader_2.54mm:PinHeader_1x08_P2.54mm_Horizontal
- J4: footprint Connector_PinHeader_2.54mm:PinHeader_1x04_P2.54mm_Vertical -> Connector_PinHeader_2.54mm:PinHeader_1x04_P2.54mm_Horizontal
Connections:
- net 3V3: now also R27.1
- net 5V: now also J3.2 (Pin_2); no longer J3.7 (Pin_7)
- net EncoderIn/ENC_A+: now also J3.8 (Pin_8); no longer J3.1 (Pin_1)
- net EncoderIn/ENC_A-: now also J3.7 (Pin_7); no longer J3.2 (Pin_2)
- net EncoderIn/ENC_B+: now also J3.6 (Pin_6); no longer J3.3 (Pin_3)
- net EncoderIn/ENC_B-: now also J3.5 (Pin_5); no longer J3.4 (Pin_4)
- net EncoderIn/ENC_Z+: now also J3.4 (Pin_4); no longer J3.5 (Pin_5)
- net EncoderIn/ENC_Z-: now also J3.3 (Pin_3); no longer J3.6 (Pin_6)
- net GND: now also J1.1 (Pin_1), J2.1 (Pin_1), J3.1 (Pin_1), SW29.2, SW30.2; no longer J1.2 (Pin_2), J2.5 (Pin_5), J3.8 (Pin_8)
- net MotorDriveOut/ALR_IN: now also J2.2 (Pin_2); no longer J2.4 (Pin_4)
- net MotorDriveOut/DIR_OUT: now also J2.4 (Pin_4); no longer J2.2 (Pin_2)
- net MotorDriveOut/STP_OUT: now also J2.5 (Pin_5); no longer J2.1 (Pin_1)
- net Power Distribution/36V: now also J1.2 (Pin_2); no longer J1.1 (Pin_1)
- net at U1.25 (IO0): now also SW29.1
- net at U1.3 (EN): now also R27.2, SW30.1
- net PROG_RX: now reaches U1.34 (RXD0/IO3)
- net PROG_TX: now reaches U1.35 (TXD0/IO1)
- no-connect marks 12 -> 8

Commit message: syncing
Parts:
- added J5: SCREEN_CONN, Connector_PinHeader_2.54mm:PinHeader_1x04_P2.54mm_Horizontal, symbol Connector:Conn_01x04_Socket
- added J6: PROG_HEADER, Connector_PinHeader_2.54mm:PinHeader_1x04_P2.54mm_Horizontal, symbol Connector:Conn_01x04_Socket
Connections:
- net 3V3: now also J5.2 (Pin_2), J6.2 (Pin_2)
- net GND: now also J5.1 (Pin_1), J6.1 (Pin_1)
- net PROG_RX: now also J6.3 (Pin_3)
- net PROG_TX: now also J6.4 (Pin_4)
- net SCREEN_CLK: now also J5.3 (Pin_3)
- net SCREEN_SDA: now also J5.4 (Pin_4)
