File: FourthAxis/EncoderIn.kicad_sch (KiCad schematic)
At the start: 0 parts

Commit message: Encoder input added?
Parts:
- added R18, R19, R20: 10k, Resistor_SMD:R_0603_1608Metric, symbol Device:R_US
- added U10, U5, U9: MAX3485, Package_SO:SOIC-8_3.9x4.9mm_P1.27mm, symbol Interface_UART:MAX3485
Connections:
- new net: R18.1, U5.2 (~{RE})
- new net: R20.1, U10.2 (~{RE})
- new net: R19.1, U9.2 (~{RE})
- new net 3V3: U10.8 (VCC), U5.8 (VCC), U9.8 (VCC)
- new net ENC_A: U5.1 (RO)
- new net ENC_A+: U5.6 (A)
- new net ENC_A-: U5.7 (B)
- new net ENC_B: U9.1 (RO)
- new net ENC_B+: U9.6 (A)
- new net ENC_B-: U9.7 (B)
- new net ENC_Z: U10.1 (RO)
- new net ENC_Z+: U10.6 (A)
- new net ENC_Z-: U10.7 (B)
- new net GND: R18.2, R19.2, R20.2, U10.5 (GND), U5.5 (GND), U9.5 (GND)

Commit message: digikey PN and footprints
Parts:
- added R22, R24, R26: 120, Resistor_SMD:R_0603_1608Metric, symbol Device:R_US
- R21: renamed from R18; digikey (none) -> 311-10.0KHRCT-ND
- R23: renamed from R19; digikey (none) -> 311-10.0KHRCT-ND
- R25: renamed from R20; digikey (none) -> 311-10.0KHRCT-ND
- U11: renamed from U5; digikey (none) -> 5272-MAX3485ESA-EVCT-ND
- U12: renamed from U9; digikey (none) -> 5272-MAX3485ESA-EVCT-ND
- U13: renamed from U10; digikey (none) -> 5272-MAX3485ESA-EVCT-ND
Connections:
- net ENC_A+: now also R22.2
- net ENC_A-: now also R22.1
- net ENC_B+: now also R24.2
- net ENC_B-: now also R24.1
- net ENC_Z+: now also R26.2
- net ENC_Z-: now also R26.1
