File: FourthAxis/EncoderIn.kicad_sch (KiCad schematic)
At the start: 13 parts, among them U11 MAX3485, U12 MAX3485, U13 MAX3485

Commit message: boards ordered
Parts:
- C11: digikey 1276-1184-1-ND -> 1292-0603X106M100CT-ND
Changed lines of the file:
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@@
 			)
 		)
-		(property "digikey" "1276-1184-1-ND"
+		(property "digikey" "1292-0603X106M100CT-ND"
 			(at 41.91 40.64 0)
 			(hide yes)
