File: FourthAxis/MotorDriveOut.kicad_sch (KiCad schematic)
At the start: 1 part, among them U8 SN74LVC1T45DBV

Commit message: shaunmotorwork
Parts:
- added R18, R19, R20: 10k, Resistor_SMD:R_0603_1608Metric, symbol Device:R_US
- added U10, U11, U9: SN74LVC1T45DBV, Package_TO_SOT_SMD:SOT-23-6, symbol Logic_LevelTranslator:SN74LVC1T45DBV
Connections:
- net 3V3: now reaches U8.1 (VCCA)
- net 3V3: now also U10.1 (VCCA), U11.1 (VCCA), U9.1 (VCCA)
- net GND: now reaches U8.2 (GND)
- net GND: now also U10.2 (GND), U11.2 (GND), U11.5 (DIR), U9.2 (GND)
- net MOTOR_STP: now reaches U8.3 (A)
- net STP_OUT: now reaches U8.4 (B)
- net at U8.5 (DIR): now also R18.2
- net 5V: now reaches U8.6 (VCCB)
- net 5V: now also R18.1, R19.1, R20.1, U10.6 (VCCB), U11.6 (VCCB), U9.6 (VCCB)
- new net: R19.2, U9.5 (DIR)
- new net: R20.2, U10.5 (DIR)
- new net ALR_IN: U11.4 (B)
- new net DIR_OUT: U9.4 (B)
- new net EN_OUT: U10.4 (B)
- new net MOTOR_ALR: U11.3 (A)
- new net MOTOR_EN: U10.3 (A)
- new net STEP_DIR: U9.3 (A)
Other:
- moved on the sheet: U8

Commit message: digikey PN and footprints
Parts:
- R18, R19, R20: digikey (none) -> 311-10.0KHRCT-ND
- U10: renamed from U11; digikey (none) -> 296-16843-1-ND
- U7: renamed from U8; digikey (none) -> 296-16843-1-ND
- U8: renamed from U9; digikey (none) -> 296-16843-1-ND
- U9: renamed from U10; digikey (none) -> 296-16843-1-ND
Changed lines of the file:
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@@
+			)
+		)
+		(property "digikey" "311-10.0KHRCT-ND"
+			(at 74.93 87.63 90)
+			(hide yes)
+			(show_name no)
+			(do_not_autoplace no)
+			(effects
+				(font
+					(size 1.27 1.27)
+				)
 			)
 		)
@@
 		(dnp no)
 		(fields_autoplaced yes)
-		(property "Reference" "U8"
+		(property "Reference" "U7"
 			(at 110.49 31.6798 0)
 			(show_name no)
@@
 		)
 		(property "Digikey" "74LVC1T45W6-7DICT-ND"
+			(at 92.71 38.1 0)
+			(hide yes)
+			(show_name no)
+			(do_not_autoplace no)
+			(effects
+				(font
+					(size 1.27 1.27)
+				)
+			)
+		)
+		(property "digikey" "296-16843-1-ND"
 			(at 92.71 38.1 0)
 			(hide yes)
@@
 			(project "FourthAxis"
 				(path "/32b0d774-33bf-42ba-9d9e-f33866433972/8b37deee-9195-4f8e-b247-4b42a620bb4c"
-					(reference "U8")
+					(reference "U7")
 					(unit 1)
 				)
@@
 		(dnp no)
 		(fields_autoplaced yes)
-		(property "Reference" "U9"
+		(property "Reference" "U8"
 			(at 110.49 76.1298 0)
 			(show_name no)
@@
 		)
 		(property "Digikey" "74LVC1T45W6-7DICT-ND"
+			(at 92.71 82.55 0)
+			(hide yes)
+			(show_name no)
+			(do_not_autoplace no)
+			(effects
+				(font
+					(size 1.27 1.27)
+				)
+			)
+		)
+		(property "digikey" "296-16843-1-ND"
 			(at 92.71 82.55 0)
 			(hide yes)
@@
 			(project "FourthAxis"
 				(path "/32b0d774-33bf-42ba-9d9e-f33866433972/8b37deee-9195-4f8e-b247-4b42a620bb4c"
-					(reference "U9")
+					(reference "U8")
 					(unit 1)
 				)
@@
 		(dnp no)
 		(fields_autoplaced yes)
-		(property "Reference" "U11"
+		(property "Reference" "U10"
 			(at 207.01 120.5798 0)
 			(show_name no)
@@
 		)
 		(property "Digikey" "74LVC1T45W6-7DICT-ND"
+			(at 189.23 127 0)
+			(hide yes)
+			(show_name no)
+			(do_not_autoplace no)
+			(effects
+				(font
+					(size 1.27 1.27)
+				)
+			)
+		)
+		(property "digikey" "296-16843-1-ND"
 			(at 189.23 127 0)
 			(hide yes)
@@
 			(project "FourthAxis"
 				(path "/32b0d774-33bf-42ba-9d9e-f33866433972/8b37deee-9195-4f8e-b247-4b42a620bb4c"
-					(reference "U11")
+					(reference "U10")
 					(unit 1)
 				)
@@
 		(dnp no)
 		(fields_autoplaced yes)
-		(property "Reference" "U10"
+		(property "Reference" "U9"
 			(at 110.49 120.5798 0)
 			(show_name no)
@@
 		)
 		(property "Digikey" "74LVC1T45W6-7DICT-ND"
+			(at 92.71 127 0)
+			(hide yes)
+			(show_name no)
+			(do_not_autoplace no)
+			(effects
+				(font
+					(size 1.27 1.27)
+				)
+			)
+		)
+		(property "digikey" "296-16843-1-ND"
 			(at 92.71 127 0)
 			(hide yes)
@@
 			(project "FourthAxis"
 				(path "/32b0d774-33bf-42ba-9d9e-f33866433972/8b37deee-9195-4f8e-b247-4b42a620bb4c"
-					(reference "U10")
+					(reference "U9")
 					(unit 1)
 				)
@@
 			)
 		)
+		(property "digikey" "311-10.0KHRCT-ND"
+			(at 74.93 132.08 90)
+			(hide yes)
+			(show_name no)
+			(do_not_autoplace no)
+			(effects
+				(font
+					(size 1.27 1.27)
+				)
+			)
+		)
 		(pin "1"
 		)
@@
 			(hide yes)
 			(show_name no)
+			(do_not_autoplace no)
+			(effects
+				(font
+					(size 1.27 1.27)
+				)
+			)
+		)
+		(property "digikey" "311-10.0KHRCT-ND"
+			(at 74.93 43.18 90)
+			(hide yes)
+			(show_name no)
