File: FourthAxis/Knobs.kicad_sch (KiCad schematic)
At the start: 7 parts, among them SW27 SW_Rotary_1x4_MP, SW28 SW_Rotary_1x3_MP

Commit message: name and layout
Parts:
- R13, R14, R15, R5, R6: footprint (none) -> Resistor_SMD:R_0603_1608Metric
Changed lines of the file:
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@@
 			)
 		)
-		(property "Footprint" ""
+		(property "Footprint" "Resistor_SMD:R_0603_1608Metric"
 			(at 115.316 66.294 90)
 			(hide yes)
@@
 			)
 		)
-		(property "Footprint" ""
+		(property "Footprint" "Resistor_SMD:R_0603_1608Metric"
 			(at 115.316 48.514 90)
 			(hide yes)
@@
 			)
 		)
-		(property "Footprint" ""
+		(property "Footprint" "Resistor_SMD:R_0603_1608Metric"
 			(at 175.006 53.594 90)
 			(hide yes)
@@
 			)
 		)
-		(property "Footprint" ""
+		(property "Footprint" "Resistor_SMD:R_0603_1608Metric"
 			(at 115.316 57.404 90)
 			(hide yes)
@@
 			)
 		)
-		(property "Footprint" ""
+		(property "Footprint" "Resistor_SMD:R_0603_1608Metric"
 			(at 175.006 62.484 90)
 			(hide yes)

Commit message: Nick end of wed
Parts:
- SW27: value SW_Rotary_1x4_MP -> MODE_SWITCH
- SW28: value SW_Rotary_1x3_MP -> MULT_SWITCH
Other:
- moved on the sheet: R13, R14, R15, R5, R6, SW27, SW28

Commit message: digikey PN and footprints
Parts:
- R13: digikey (none) -> 311-10.0KHRCT-ND
- R14: renamed from R6; digikey (none) -> 311-10.0KHRCT-ND
- R15: renamed from R5; digikey (none) -> 311-10.0KHRCT-ND
- R16: renamed from R14; digikey (none) -> 311-10.0KHRCT-ND
- R17: renamed from R15; digikey (none) -> 311-10.0KHRCT-ND
- SW27: footprint (none) -> Connector_PinHeader_2.54mm:PinHeader_1x05_P2.54mm_Vertical
- SW28: footprint (none) -> Connector_PinHeader_2.54mm:PinHeader_1x04_P2.54mm_Vertical
Changed lines of the file:
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@@
 		(dnp no)
 		(fields_autoplaced yes)
-		(property "Reference" "R5"
+		(property "Reference" "R15"
 			(at 87.63 71.1199 0)
 			(show_name no)
@@
 		)
 		(property "Description" "Resistor, US symbol"
+			(at 85.09 72.39 0)
+			(hide yes)
+			(show_name no)
+			(do_not_autoplace no)
+			(effects
+				(font
+					(size 1.27 1.27)
+				)
+			)
+		)
+		(property "digikey" "311-10.0KHRCT-ND"
 			(at 85.09 72.39 0)
 			(hide yes)
@@
 			(project "FourthAxis"
 				(path "/32b0d774-33bf-42ba-9d9e-f33866433972/b72fb8ef-4cdc-46b5-9289-178b699f5f8c"
-					(reference "R5")
+					(reference "R15")
 					(unit 1)
 				)
@@
 			)
 		)
+		(property "digikey" "311-10.0KHRCT-ND"
+			(at 85.09 54.61 0)
+			(hide yes)
+			(show_name no)
+			(do_not_autoplace no)
+			(effects
+				(font
+					(size 1.27 1.27)
+				)
+			)
+		)
 		(pin "1"
 		)
@@
 		(dnp no)
 		(fields_autoplaced yes)
-		(property "Reference" "R14"
+		(property "Reference" "R16"
 			(at 147.32 58.4199 0)
 			(show_name no)
@@
 		)
 		(property "Description" "Resistor, US symbol"
+			(at 144.78 59.69 0)
+			(hide yes)
+			(show_name no)
+			(do_not_autoplace no)
+			(effects
+				(font
+					(size 1.27 1.27)
+				)
+			)
+		)
+		(property "digikey" "311-10.0KHRCT-ND"
 			(at 144.78 59.69 0)
 			(hide yes)
@@
 			(project "FourthAxis"
 				(path "/32b0d774-33bf-42ba-9d9e-f33866433972/b72fb8ef-4cdc-46b5-9289-178b699f5f8c"
-					(reference "R14")
+					(reference "R16")
 					(unit 1)
 				)
@@
 			)
 		)
-		(property "Footprint" ""
+		(property "Footprint" "Connector_PinHeader_2.54mm:PinHeader_1x05_P2.54mm_Vertical"
 			(at 59.69 74.93 0)
 			(hide yes)
@@
 		(dnp no)
 		(fields_autoplaced yes)
-		(property "Reference" "R6"
+		(property "Reference" "R14"
 			(at 87.63 62.2299 0)
 			(show_name no)
@@
 		)
 		(property "Description" "Resistor, US symbol"
+			(at 85.09 63.5 0)
+			(hide yes)
+			(show_name no)
+			(do_not_autoplace no)
+			(effects
+				(font
+					(size 1.27 1.27)
+				)
+			)
+		)
+		(property "digikey" "311-10.0KHRCT-ND"
 			(at 85.09 63.5 0)
 			(hide yes)
@@
 			(project "FourthAxis"
 				(path "/32b0d774-33bf-42ba-9d9e-f33866433972/b72fb8ef-4cdc-46b5-9289-178b699f5f8c"
-					(reference "R6")
+					(reference "R14")
 					(unit 1)
 				)
@@
 		(dnp no)
 		(fields_autoplaced yes)
-		(property "Reference" "R15"
+		(property "Reference" "R17"
 			(at 147.32 67.3099 0)
 			(show_name no)
@@
 		)
 		(property "Description" "Resistor, US symbol"
+			(at 144.78 68.58 0)
+			(hide yes)
+			(show_name no)
+			(do_not_autoplace no)
+			(effects
+				(font
+					(size 1.27 1.27)
+				)
+			)
+		)
+		(property "digikey" "311-10.0KHRCT-ND"
 			(at 144.78 68.58 0)
 			(hide yes)
@@
 			(project "FourthAxis"
 				(path "/32b0d774-33bf-42ba-9d9e-f33866433972/b72fb8ef-4cdc-46b5-9289-178b699f5f8c"
-					(reference "R15")
+					(reference "R17")
 					(unit 1)
 				)
@@
 			)
 		)
-		(property "Footprint" ""
+		(property "Footprint" "Connector_PinHeader_2.54mm:PinHeader_1x04_P2.54mm_Vertical"
 			(at 119.38 72.39 0)
 			(hide yes)

Commit message: Layout work
Parts:
- SW27: footprint Connector_PinHeader_2.54mm:PinHeader_1x05_P2.54mm_Vertical -> Connector_PinHeader_2.54mm:PinHeader_1x05_P2.54mm_Horizontal
- SW28: footprint Connector_PinHeader_2.54mm:PinHeader_1x04_P2.54mm_Vertical -> Connector_PinHeader_2.54mm:PinHeader_1x04_P2.54mm_Horizontal
Changed lines of the file:
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@@
 			)
 		)
-		(property "Footprint" "Connector_PinHeader_2.54mm:PinHeader_1x05_P2.54mm_Vertical"
+		(property "Footprint" "Connector_PinHeader_2.54mm:PinHeader_1x05_P2.54mm_Horizontal"
 			(at 59.69 74.93 0)
 			(hide yes)
@@
 			)
 		)
-		(property "Footprint" "Connector_PinHeader_2.54mm:PinHeader_1x04_P2.54mm_Vertical"
+		(property "Footprint" "Connector_PinHeader_2.54mm:PinHeader_1x04_P2.54mm_Horizontal"
 			(at 119.38 72.39 0)
 			(hide yes)
