File: FourthAxis/Knobs.kicad_sch (KiCad schematic)
At the start: 7 parts, among them SW27 MODE_SWITCH, SW28 MULT_SWITCH

Commit message: BOM export
Parts:
- SW27, SW28: now left out of the parts list
Changed lines of the file:
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@@
 		(body_style 1)
 		(exclude_from_sim no)
-		(in_bom yes)
+		(in_bom no)
 		(on_board yes)
 		(in_pos_files yes)
@@
 		(body_style 1)
 		(exclude_from_sim no)
-		(in_bom yes)
-		(on_board yes)
-		(in_pos_files yes)
+		(in_bom no)
+		(on_board yes)
+		(in_pos_files yes)
