File: FourthAxis/FourthAxis.kicad_pcb (KiCad board)
At the start: 2 copper layers, 64 parts, among them SW1 SW_Push, SW10 SW_Push, SW11 SW_Push, SW12 SW_Push, SW13 SW_Push, SW14 SW_Push, SW15 SW_Push, SW16 SW_Push, SW17 SW_Push, SW18 SW_Push, SW19 SW_Push, SW2 SW_Push, SW20 SW_Push, SW21 SW_Push, SW22 SW_Push, SW23 SW_Push, SW24 SW_Push, SW25 SW_Push, SW26 SW_Push, SW3 SW_Push, SW4 SW_Push, SW5 SW_Push, SW6 SW_Push, SW7 SW_Push, SW8 SW_Push, SW9 SW_Push, U1 ESP32-WROOM-32, U2 74HC237, U3 XL1509-5.0, U4 XL1509-3.3

Commit message: name and layout
Parts:
- added R11: 10k, Resistor_SMD:R_0603_1608Metric, F.Cu at (223.7, 115.6)
- added R12: 10k, Resistor_SMD:R_0603_1608Metric, F.Cu at (223.7, 118.1)
- added R13: 10k, Resistor_SMD:R_0603_1608Metric, F.Cu at (217.7, 120.6)
- added R14: 10k, Resistor_SMD:R_0603_1608Metric, F.Cu at (217.7, 123.1)
- added R15: 10k, Resistor_SMD:R_0603_1608Metric, F.Cu at (217.7, 125.6)
- added R5: 10k, Resistor_SMD:R_0603_1608Metric, F.Cu at (217.7, 115.6)
- added R6: 10k, Resistor_SMD:R_0603_1608Metric, F.Cu at (217.7, 118.1)
- added U6: SN74LVC1T45DBV, Package_TO_SOT_SMD:SOT-23-6, F.Cu at (214.4, 137.1)
- added U7: SN74LVC1T45DBV, Package_TO_SOT_SMD:SOT-23-6, F.Cu at (214.4, 141.7)
- SW1: value SW_Push -> NUM_1; footprint Button_Switch_Keyboard:SW_Cherry_MX_1.00u_PCB -> CustomFooties:SW_Cherry_MX_1.00u_PCB
- SW10: value SW_Push -> NUM_6; footprint Button_Switch_Keyboard:SW_Cherry_MX_1.00u_PCB -> CustomFooties:SW_Cherry_MX_1.00u_PCB
- SW11: value SW_Push -> NUM_9; footprint Button_Switch_Keyboard:SW_Cherry_MX_1.00u_PCB -> CustomFooties:SW_Cherry_MX_1.00u_PCB
- SW12: value SW_Push -> PLUS_MINUS; footprint Button_Switch_Keyboard:SW_Cherry_MX_1.00u_PCB -> CustomFooties:SW_Cherry_MX_1.00u_PCB
- SW13: value SW_Push -> DELETE; footprint Button_Switch_Keyboard:SW_Cherry_MX_1.00u_PCB -> CustomFooties:SW_Cherry_MX_1.00u_PCB
- SW14: value SW_Push -> ENTER; footprint Button_Switch_Keyboard:SW_Cherry_MX_1.00u_PCB -> CustomFooties:SW_Cherry_MX_1.00u_PCB
- SW15: value SW_Push -> SET_ZERO; footprint Button_Switch_Keyboard:SW_Cherry_MX_1.00u_PCB -> CustomFooties:SW_Cherry_MX_1.00u_PCB
- SW16: value SW_Push -> SET_SPLN; footprint Button_Switch_Keyboard:SW_Cherry_MX_1.00u_PCB -> CustomFooties:SW_Cherry_MX_1.00u_PCB
- SW17: value SW_Push -> ANG_ABS; footprint Button_Switch_Keyboard:SW_Cherry_MX_1.00u_PCB -> CustomFooties:SW_Cherry_MX_1.00u_PCB
- SW18: value SW_Push -> ROT_CCW; footprint Button_Switch_Keyboard:SW_Cherry_MX_1.00u_PCB -> CustomFooties:SW_Cherry_MX_1.00u_PCB
- SW19: value SW_Push -> RET_ZERO; footprint Button_Switch_Keyboard:SW_Cherry_MX_1.00u_PCB -> CustomFooties:SW_Cherry_MX_1.00u_PCB
- SW2: value SW_Push -> NUM_4; footprint Button_Switch_Keyboard:SW_Cherry_MX_1.00u_PCB -> CustomFooties:SW_Cherry_MX_1.00u_PCB
- SW20: value SW_Push -> NXT_SPLN; footprint Button_Switch_Keyboard:SW_Cherry_MX_1.00u_PCB -> CustomFooties:SW_Cherry_MX_1.00u_PCB
- SW21: value SW_Push -> ANG_INC; footprint Button_Switch_Keyboard:SW_Cherry_MX_1.00u_PCB -> CustomFooties:SW_Cherry_MX_1.00u_PCB
- SW22: value SW_Push -> ROT_CW; footprint Button_Switch_Keyboard:SW_Cherry_MX_1.00u_PCB -> CustomFooties:SW_Cherry_MX_1.00u_PCB
- SW23: value SW_Push -> EXTRA_1; footprint Button_Switch_Keyboard:SW_Cherry_MX_1.00u_PCB -> CustomFooties:SW_Cherry_MX_1.00u_PCB
- SW24: value SW_Push -> EXTRA_2; footprint Button_Switch_Keyboard:SW_Cherry_MX_1.00u_PCB -> CustomFooties:SW_Cherry_MX_1.00u_PCB
- SW25: value SW_Push -> EXTRA_3; footprint Button_Switch_Keyboard:SW_Cherry_MX_1.00u_PCB -> CustomFooties:SW_Cherry_MX_1.00u_PCB
- SW26: value SW_Push -> EXTRA_4; footprint Button_Switch_Keyboard:SW_Cherry_MX_1.00u_PCB -> CustomFooties:SW_Cherry_MX_1.00u_PCB
- SW3: value SW_Push -> NUM_7; footprint Button_Switch_Keyboard:SW_Cherry_MX_1.00u_PCB -> CustomFooties:SW_Cherry_MX_1.00u_PCB
- SW4: value SW_Push -> DECIMAL; footprint Button_Switch_Keyboard:SW_Cherry_MX_1.00u_PCB -> CustomFooties:SW_Cherry_MX_1.00u_PCB
- SW5: value SW_Push -> NUM_2; footprint Button_Switch_Keyboard:SW_Cherry_MX_1.00u_PCB -> CustomFooties:SW_Cherry_MX_1.00u_PCB
- SW6: value SW_Push -> NUM_5; footprint Button_Switch_Keyboard:SW_Cherry_MX_1.00u_PCB -> CustomFooties:SW_Cherry_MX_1.00u_PCB
- SW7: value SW_Push -> NUM_8; footprint Button_Switch_Keyboard:SW_Cherry_MX_1.00u_PCB -> CustomFooties:SW_Cherry_MX_1.00u_PCB
- SW8: value SW_Push -> NUM_0; footprint Button_Switch_Keyboard:SW_Cherry_MX_1.00u_PCB -> CustomFooties:SW_Cherry_MX_1.00u_PCB
- SW9: value SW_Push -> NUM_3; footprint Button_Switch_Keyboard:SW_Cherry_MX_1.00u_PCB -> CustomFooties:SW_Cherry_MX_1.00u_PCB
- moved SW4 214.0 mm to (54.6, 141.5)
- moved SW3 213.7 mm to (54.6, 122.2)
- moved SW2 213.5 mm to (54.6, 102.9)
- moved SW8 211.5 mm to (73.9, 141.5)
- moved SW7 210.9 mm to (73.9, 122.2)
- moved SW12 210.3 mm to (93.2, 141.5)
- moved SW5 201.9 mm to (73.9, 83.6)
- moved SW6 200.7 mm to (73.9, 102.9)
- moved SW9 194.1 mm to (93.2, 83.6)
- moved SW10 193.3 mm to (93.2, 102.9)
- moved SW11 192.5 mm to (93.2, 122.2)
- moved SW14 186.4 mm to (112.5, 141.5)
- moved SW13 186.0 mm to (112.5, 122.2)
- moved SW18 184.2 mm to (131.8, 141.5)
- moved SW17 183.5 mm to (131.8, 122.2)
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Connections:
- U1 pad 10: KEY_7 -> KNOB_2
- U1 pad 24: KNOB_1 -> unconnected-(U1-IO2-Pad24)
- U1 pad 26: KNOB_2 -> HAND_INT
- U1 pad 34: HAND_INT -> unconnected-(U1-RXD0/IO3-Pad34)
- U1 pad 37: KEY_6 -> KNOB_1

Commit message: digikey PN and footprints
Parts:
- added C1: 470u, Capacitor_THT:C_Radial_D10.0mm_H20.0mm_P5.00mm, F.Cu at (269.5, 84.8)
- added C2: 1u, Capacitor_SMD:C_0603_1608Metric, F.Cu at (297.5, 96.0)
- added C3: 330u, Capacitor_SMD:CP_Elec_6.3x7.7, F.Cu at (300.5, 82.3)
- added C4: 470u, Capacitor_THT:C_Radial_D10.0mm_H20.0mm_P5.00mm, F.Cu at (269.6, 105.4)
- added C5: 1u, Capacitor_SMD:C_0603_1608Metric, F.Cu at (297.5, 99.0)
- added C6: 330u, Capacitor_SMD:CP_Elec_6.3x7.7, F.Cu at (300.5, 90.4)
- added D27: 1N5821, Diode_SMD:D_SOD-123, F.Cu at (282.9, 110.1)
- added D28: 1N5821, Diode_SMD:D_SOD-123, F.Cu at (282.9, 116.8)
- added J1: 36V POWER IN, Connector_PinHeader_2.54mm:PinHeader_1x02_P2.54mm_Vertical, F.Cu at (314.6, 95.2)
- added J2: DRIVER_CONN, Connector_PinHeader_2.54mm:PinHeader_1x05_P2.54mm_Vertical, F.Cu at (314.6, 80.5)
- added J3: ENC_CONN, Connector_PinHeader_2.54mm:PinHeader_1x08_P2.54mm_Vertical, F.Cu at (310.0, 80.5)
- added J4: HW_CONN, Connector_PinHeader_2.54mm:PinHeader_1x04_P2.54mm_Vertical, F.Cu at (319.2, 80.5)
- added L1: 68u, Inductor_SMD:L_12x12mm_H6mm, F.Cu at (287.9, 85.3)
- added L2: 47u, Inductor_SMD:L_12x12mm_H6mm, F.Cu at (287.9, 99.6)
- added R11: 10k, Resistor_SMD:R_0603_1608Metric, F.Cu at (301.2, 95.5)
- added R12: 10k, Resistor_SMD:R_0603_1608Metric, F.Cu at (301.2, 97.5)
- added R18: 10k, Resistor_SMD:R_0603_1608Metric, F.Cu at (280.0, 123.4)
- added R19: 10k, Resistor_SMD:R_0603_1608Metric, F.Cu at (280.0, 126.0)
- added R20: 10k, Resistor_SMD:R_0603_1608Metric, F.Cu at (280.0, 128.5)
- added R21: 10k, Resistor_SMD:R_0603_1608Metric, F.Cu at (268.8, 123.4)
- added R22: 120, Resistor_SMD:R_0603_1608Metric, F.Cu at (268.8, 126.0)
- added R23: 10k, Resistor_SMD:R_0603_1608Metric, F.Cu at (268.8, 128.5)
- added R24: 120, Resistor_SMD:R_0603_1608Metric, F.Cu at (268.8, 131.0)
- added R25: 10k, Resistor_SMD:R_0603_1608Metric, F.Cu at (268.8, 133.5)
- added R26: 120, Resistor_SMD:R_0603_1608Metric, F.Cu at (268.8, 136.0)
- added SW27: MODE_SWITCH, Connector_PinHeader_2.54mm:PinHeader_1x05_P2.54mm_Vertical, F.Cu at (286.3, 124.5)
- added SW28: MULT_SWITCH, Connector_PinHeader_2.54mm:PinHeader_1x04_P2.54mm_Vertical, F.Cu at (290.9, 124.5)
- added U10: SN74LVC1T45DBV, Package_TO_SOT_SMD:SOT-23-6, F.Cu at (275.4, 138.5)
- added U11: MAX3485, Package_SO:SOIC-8_3.9x4.9mm_P1.27mm, F.Cu at (262.6, 125.6)
- added U12: MAX3485, Package_SO:SOIC-8_3.9x4.9mm_P1.27mm, F.Cu at (262.6, 132.1)
- added U13: MAX3485, Package_SO:SOIC-8_3.9x4.9mm_P1.27mm, F.Cu at (262.6, 138.7)
- added U7: SN74LVC1T45DBV, Package_TO_SOT_SMD:SOT-23-6, F.Cu at (275.4, 124.6)
- added U8: SN74LVC1T45DBV, Package_TO_SOT_SMD:SOT-23-6, F.Cu at (275.4, 129.2)
- added U9: SN74LVC1T45DBV, Package_TO_SOT_SMD:SOT-23-6, F.Cu at (275.4, 133.8)
- D1, D10, D11, D12, D13, D14, D15, D16, D17, D18, D19, D2, D20, D21, D22, D23, D24, D25, D26, D3, D4, D5, D6, D7, D8, D9: footprint Diode_SMD:D_SOD-323 -> Diode_SMD:D_SOD-123
- moved D1 5.61 mm to (197.6, 94.0)
- renumbered R9 to R1, R12 to R10, R6 to R14, R5 to R15, R14 to R16, R15 to R17, R8 to R2, R7 to R3, R1 to R4, R10 to R5, R2 to R6, R3 to R7, R4 to R8, R11 to R9, U6 to U3, U7 to U4, U3 to U5, U4 to U6
Connections:
- U3 pad 3: HAND_INC_A -> /HandWheel/ENC_A_IN
- U4 pad 3: HAND_INC_B -> /HandWheel/ENC_B_IN
- U5 pad 1: unconnected-(U3-VIN-Pad1) -> /Power Distribution/36V
- U5 pad 2: unconnected-(U3-OUT-Pad2) -> Net-(D27-K)
- U5 pad 3: unconnected-(U3-FB-Pad3) -> 5V
- U5 pad 4: unconnected-(U3-~{EN}-Pad4) -> Net-(U5-~{EN})
- U5 pad 5: Net-(U3-GND-Pad5) -> GND
- U5 pad 6: Net-(U3-GND-Pad5) -> GND
- U5 pad 7: Net-(U3-GND-Pad5) -> GND
- U5 pad 8: Net-(U3-GND-Pad5) -> GND
- U6 pad 1: unconnected-(U4-VIN-Pad1) -> /Power Distribution/36V
- U6 pad 2: unconnected-(U4-OUT-Pad2) -> Net-(D28-K)
- U6 pad 3: unconnected-(U4-FB-Pad3) -> 3V3
- U6 pad 4: unconnected-(U4-~{EN}-Pad4) -> Net-(U6-~{EN})
- U6 pad 5: Net-(U4-GND-Pad5) -> GND
- U6 pad 6: Net-(U4-GND-Pad5) -> GND
- U6 pad 7: Net-(U4-GND-Pad5) -> GND
- U6 pad 8: Net-(U4-GND-Pad5) -> GND

Commit message: Layout work
Parts:
- added R27: 10k, Resistor_SMD:R_0603_1608Metric, F.Cu at (49.8, 71.1)
- added SW29: BOOT, Button_Switch_SMD:SW_Push_1P1T_NO_CK_KMR2, F.Cu at (44.5, 66.8)
- added SW30: RESET, Button_Switch_SMD:SW_Push_1P1T_NO_CK_KMR2, F.Cu at (44.5, 73.2)
- J1: footprint Connector_PinHeader_2.54mm:PinHeader_1x02_P2.54mm_Vertical -> Connector_PinHeader_2.54mm:PinHeader_1x02_P2.54mm_Horizontal
- J2, SW27: footprint Connector_PinHeader_2.54mm:PinHeader_1x05_P2.54mm_Vertical -> Connector_PinHeader_2.54mm:PinHeader_1x05_P2.54mm_Horizontal
- J3: footprint Connector_PinHeader_2.54mm:PinHeader_1x08_P2.54mm_Vertical -> Connector_PinHeader_2.54mm:PinHeader_1x08_P2.54mm_Horizontal
- J4, SW28: footprint Connector_PinHeader_2.54mm:PinHeader_1x04_P2.54mm_Vertical -> Connector_PinHeader_2.54mm:PinHeader_1x04_P2.54mm_Horizontal
- moved J1 272.2 mm to (44.4, 62.0), turned to 90 degrees
- moved SW28 247.1 mm to (51.8, 62.0), turned to 90 degrees
- moved J2 236.1 mm to (79.2, 62.0), turned to 90 degrees
- moved SW27 230.7 mm to (64.3, 62.0), turned to 90 degrees
- moved R18 210.2 mm to (77.5, 66.9), turned to 90 degrees
- moved R19 208.5 mm to (80.1, 66.9), turned to 90 degrees
- moved R20 206.8 mm to (82.6, 66.9), turned to 90 degrees
- moved U7 203.8 mm to (78.7, 71.5), turned to 90 degrees
- moved U8 200.6 mm to (83.3, 71.5), turned to 90 degrees
- moved U9 197.6 mm to (87.9, 71.5), turned to 90 degrees
- moved U10 194.7 mm to (92.6, 71.5), turned to 90 degrees
- moved J4 174.9 mm to (145.3, 62.0), turned to 90 degrees
- moved R16 174.8 mm to (52.9, 64.8)
- moved R17 172.8 mm to (55.9, 64.8)
- moved R13 162.1 mm to (65.3, 65.3), turned to -90 degrees
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Connections:
- J1 pad 1: /Power Distribution/36V -> GND
- J1 pad 2: GND -> /Power Distribution/36V
- J2 pad 1: /MotorDriveOut/STP_OUT -> GND
- J2 pad 2: /MotorDriveOut/DIR_OUT -> /MotorDriveOut/ALR_IN
- J2 pad 4: /MotorDriveOut/ALR_IN -> /MotorDriveOut/DIR_OUT
- J2 pad 5: GND -> /MotorDriveOut/STP_OUT
- J3 pad 1: /EncoderIn/ENC_A+ -> GND
- J3 pad 2: /EncoderIn/ENC_A- -> 5V
- J3 pad 3: /EncoderIn/ENC_B+ -> /EncoderIn/ENC_Z-
- J3 pad 4: /EncoderIn/ENC_B- -> /EncoderIn/ENC_Z+
- J3 pad 5: /EncoderIn/ENC_Z+ -> /EncoderIn/ENC_B-
- J3 pad 6: /EncoderIn/ENC_Z- -> /EncoderIn/ENC_B+
- J3 pad 7: 5V -> /EncoderIn/ENC_A-
- J3 pad 8: GND -> /EncoderIn/ENC_A+
- U1 pad 25: unconnected-(U1-IO0-Pad25) -> Net-(U1-IO0)
- U1 pad 3: unconnected-(U1-EN-Pad3) -> Net-(U1-EN)
- U1 pad 34: unconnected-(U1-RXD0/IO3-Pad34) -> PROG_RX
- U1 pad 35: unconnected-(U1-TXD0/IO1-Pad35) -> PROG_TX
Other:
- board outline added: 135.1 x 104.9 mm

Commit message: syncing
Parts:
- added J5: SCREEN_CONN, Connector_PinHeader_2.54mm:PinHeader_1x04_P2.54mm_Horizontal, F.Cu at (387.9, 95.0)
- added J6: PROG_HEADER, Connector_PinHeader_2.54mm:PinHeader_1x04_P2.54mm_Horizontal, F.Cu at (387.9, 107.2)
- moved C1 178.8 mm to (417.6, 36.3)
- moved C2 178.8 mm to (445.6, 47.5)
- moved C3 178.8 mm to (448.6, 33.8)
- moved C5 178.8 mm to (446.9, 78.7)
- moved C6 178.8 mm to (449.9, 70.1)
- moved D27 178.8 mm to (431.0, 61.6)
- moved D28 178.8 mm to (432.2, 96.5)
- moved L1 178.8 mm to (436.0, 36.8)
- moved L2 178.8 mm to (437.3, 79.2)
- moved R11 178.8 mm to (449.3, 47.0)
- moved R12 178.8 mm to (450.5, 77.2)
- moved U5 178.8 mm to (415.5, 46.0)
- moved U6 178.8 mm to (421.6, 96.0)
- moved C4 178.8 mm to (419.0, 85.1)

Commit message: Layout work, added power LEDs
Parts:
- removed C1: 470u, Capacitor_THT:C_Radial_D10.0mm_H20.0mm_P5.00mm
- added C10: 1u, Capacitor_SMD:C_0603_1608Metric, F.Cu at (156.6, 52.1)
- added C11: 10u, Capacitor_SMD:C_0603_1608Metric, F.Cu at (155.1, 52.1)
- added C12: 1u, Capacitor_SMD:C_0603_1608Metric, F.Cu at (163.7, 52.1)
- added C13: 1u, Capacitor_SMD:C_0603_1608Metric, F.Cu at (170.8, 52.1)
- added C14: 1u, Capacitor_SMD:C_0603_1608Metric, F.Cu at (147.9, 54.3)
- added C15: 1u, Capacitor_SMD:C_0603_1608Metric, F.Cu at (146.4, 54.3)
- added C16: 1u, Capacitor_SMD:C_0603_1608Metric, F.Cu at (153.3, 54.3)
- added C17: 1u, Capacitor_SMD:C_0603_1608Metric, F.Cu at (151.8, 54.3)
- added C18: 1u, Capacitor_SMD:C_0603_1608Metric, F.Cu at (117.1, 82.8)
- added C19: 1u, Capacitor_SMD:C_0603_1608Metric, F.Cu at (117.1, 81.3)
- added C20: 1u, Capacitor_SMD:C_0603_1608Metric, F.Cu at (96.0, 73.4)
- added C21: 1u, Capacitor_SMD:C_0603_1608Metric, F.Cu at (96.0, 71.9)
- added C22: 1u, Capacitor_SMD:C_0603_1608Metric, F.Cu at (96.0, 62.0)
- added C23: 1u, Capacitor_SMD:C_0603_1608Metric, F.Cu at (96.0, 60.5)
- added C24: 1u, Capacitor_SMD:C_0603_1608Metric, F.Cu at (96.0, 67.8)
- added C25: 1u, Capacitor_SMD:C_0603_1608Metric, F.Cu at (96.0, 66.3)
- added C26: 1u, Capacitor_SMD:C_0603_1608Metric, F.Cu at (95.9, 55.6)
- added C27: 1u, Capacitor_SMD:C_0603_1608Metric, F.Cu at (95.9, 54.1)
- added C28: 10u, Capacitor_SMD:C_0603_1608Metric, F.Cu at (51.7, 50.8)
- added C29: 10u, Capacitor_SMD:C_0603_1608Metric, F.Cu at (51.7, 49.3)
- added C30: 1u, Capacitor_SMD:C_0603_1608Metric, F.Cu at (51.7, 47.8)
- added C7: 1u, Capacitor_SMD:C_0603_1608Metric, F.Cu at (106.2, 44.2)
- added C8: 1u, Capacitor_SMD:C_0603_1608Metric, F.Cu at (104.6, 44.2)
- added C9: 10u, Capacitor_SMD:C_0603_1608Metric, F.Cu at (103.1, 44.2)
- added D29: 36V, LED_SMD:LED_0603_1608Metric, F.Cu at (46.5, 63.9)
- added D30: 5V, LED_SMD:LED_0603_1608Metric, F.Cu at (46.5, 70.0)
- added D31: 3V3, LED_SMD:LED_0603_1608Metric, F.Cu at (46.5, 76.1)
- added D32: 1N5821, Diode_SMD:D_SOD-123, F.Cu at (45.6, 47.0)
- added H1: GND_hole, MountingHole:MountingHole_2.2mm_M2_Pad, F.Cu at (158.2, 136.9)
- added H2: GND_hole, MountingHole:MountingHole_2.2mm_M2_Pad, F.Cu at (119.6, 136.9)
- added H3: GND_hole, MountingHole:MountingHole_2.2mm_M2_Pad, F.Cu at (100.3, 136.9)
- added H4: GND_hole, MountingHole:MountingHole_2.2mm_M2_Pad, F.Cu at (61.7, 136.9)
- added H5: GND_hole, MountingHole:MountingHole_2.2mm_M2_Pad, F.Cu at (158.2, 98.3)
- added H6: GND_hole, MountingHole:MountingHole_2.2mm_M2_Pad, F.Cu at (119.6, 98.3)
- added H7: GND_hole, MountingHole:MountingHole_2.2mm_M2_Pad, F.Cu at (100.3, 98.3)
- added H8: GND_hole, MountingHole:MountingHole_2.2mm_M2_Pad, F.Cu at (61.7, 98.3)
- added R28: 10k, Resistor_SMD:R_0603_1608Metric, F.Cu at (45.7, 61.5)
- added R29: 1k, Resistor_SMD:R_0603_1608Metric, F.Cu at (45.7, 67.6)
- added R30: 1k, Resistor_SMD:R_0603_1608Metric, F.Cu at (45.7, 73.7)
- added R31: 10k, Resistor_SMD:R_0603_1608Metric, F.Cu at (47.2, 61.5)
- added R32: 1k, Resistor_SMD:R_0603_1608Metric, F.Cu at (47.2, 67.6)
- added R33: 1k, Resistor_SMD:R_0603_1608Metric, F.Cu at (47.2, 73.7)
- added R34: 1k, Resistor_SMD:R_0603_1608Metric, F.Cu at (48.8, 73.7)
- C4: value 470u -> 330u; footprint Capacitor_THT:C_Radial_D10.0mm_H20.0mm_P5.00mm -> Capacitor_SMD:CP_Elec_6.3x7.7
- J1: value 36V POWER IN -> 36V; footprint Connector_PinHeader_2.54mm:PinHeader_1x02_P2.54mm_Horizontal -> Connector_PinHeader_2.54mm:PinHeader_1x02_P2.54mm_Vertical
- J2, SW27: footprint Connector_PinHeader_2.54mm:PinHeader_1x05_P2.54mm_Horizontal -> Connector_PinHeader_2.54mm:PinHeader_1x05_P2.54mm_Vertical
- J3: footprint Connector_PinHeader_2.54mm:PinHeader_1x08_P2.54mm_Horizontal -> Connector_PinHeader_2.54mm:PinHeader_1x08_P2.54mm_Vertical
- J4, J5, J6, SW28: footprint Connector_PinHeader_2.54mm:PinHeader_1x04_P2.54mm_Horizontal -> Connector_PinHeader_2.54mm:PinHeader_1x04_P2.54mm_Vertical
- moved C2 392.6 mm to (53.2, 59.3), turned to 90 degrees
- moved R11 389.0 mm to (60.5, 59.4), turned to -90 degrees
- moved C3 384.5 mm to (64.9, 58.5), turned to 90 degrees
- moved C5 377.3 mm to (70.1, 59.1), turned to 90 degrees
- moved L1 376.4 mm to (61.1, 70.2)
- moved D27 374.2 mm to (56.8, 62.5)
- moved C4 373.8 mm to (46.5, 53.1), turned to -90 degrees
- moved R12 373.5 mm to (77.5, 59.6), turned to -90 degrees
- moved C6 368.1 mm to (81.9, 58.5), turned to 90 degrees
- moved L2 360.4 mm to (77.0, 70.2)
- moved D28 360.2 mm to (73.7, 62.4)
- moved U5 358.8 mm to (56.9, 57.5), turned to 90 degrees
- moved U6 350.0 mm to (73.8, 57.4), turned to 90 degrees
- moved J5 258.0 mm to (135.0, 43.8), turned to 90 degrees
- moved J6 257.2 mm to (135.4, 58.0), turned to 180 degrees
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Connections:
- C5 pad 1: /Power Distribution/36V -> 5V
- U6 pad 1: /Power Distribution/36V -> 5V
Other:
- board size 135.1 x 104.9 mm -> 135.1 x 114.3 mm

Commit message: started routing
Parts:
- moved R4 6.17 mm to (121.4, 64.9), turned to -90 degrees
- moved C22 5.83 mm to (96.0, 67.8)
- moved C23 5.83 mm to (96.0, 66.3)
- moved R19 5.83 mm to (96.0, 64.8)
- moved U8 5.83 mm to (99.4, 66.3)
- moved C24 5.59 mm to (96.0, 62.2)
- moved C25 5.59 mm to (96.0, 60.7)
- moved R20 5.59 mm to (96.0, 59.2)
- moved U9 5.59 mm to (99.4, 60.7)
- moved J6 2.55 mm to (137.9, 57.8)
- moved R6 2.29 mm to (129.7, 59.9)
- moved SW30 2.05 mm to (98.8, 45.8)
- moved SW29 1.55 mm to (133.3, 66.2), turned to 90 degrees
- moved C7 1.26 mm to (105.7, 45.4)
- moved C8 1.26 mm to (104.1, 45.4)
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Connections:
- net PROG_RX renamed PROG_N
- net PROG_TX renamed PROG_P
Routing:
- net KEY_4: track 0.00 -> 243.1 mm, vias 0 -> 2
- net KEY_3: track 0.00 -> 221.6 mm, vias 0 -> 2
- net KEY_2: track 0.00 -> 197.1 mm, vias 0 -> 4
- net KEY_1: track 0.00 -> 174.9 mm, vias 0 -> 3
- net Net-(U2-Y0): track 0.00 -> 147.6 mm
- net Net-(U2-Y1): track 0.00 -> 127.1 mm
- net Net-(U2-Y6): track 0.00 -> 115.4 mm
- net Net-(U2-Y2): track 0.00 -> 106.9 mm
- net Net-(U2-Y5): track 0.00 -> 91.1 mm
- net GND: track 0.00 -> 90.2 mm, vias 0 -> 65
- net Net-(U2-Y4): track 0.00 -> 68.9 mm
- net Net-(U2-Y3): track 0.00 -> 59.3 mm
- net /MotorDriveOut/STP_OUT: track 0.00 -> 36.4 mm
- net /MotorDriveOut/DIR_OUT: track 0.00 -> 32.6 mm
- net KEY_C: track 0.00 -> 31.6 mm
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Other:
- board text added: "36V"
- board text added: "3V3"
- board text added: "5V"
- board text added: "ALR"
- board text added: "DIR"
- board text added: "EN"
- board text added: "ENCA+"
- board text added: "ENCA-"
- board text added: "ENCB+"
- board text added: "ENCZ+"
- board text added: "ENCZ-"
- board text added: "GND"
- board text added: "HND_A"
- board text added: "HND_B"
- board text added: "KNOB1"
- board text added: "KNOB2"
- board text added: "MODE_2"
- board text added: "MODE_3"
- board text added: "MULT_2"
- board text added: "PROG_RX"
- board text added: "PROG_TX"
- board text added: "SCLK"
- board text added: "SDA"
- board text added: "STP"
