File: FourthAxis/FourthAxis.kicad_pcb (KiCad board)
At the start: 2 copper layers, 135.1 x 114.3 mm, 156 parts, among them J1 36V, J2 DRIVER_CONN, J3 ENC_CONN, J4 HW_CONN, J5 SCREEN_CONN, J6 PROG_HEADER, J7 ESTOP, SW1 NUM_1, SW10 NUM_6, SW11 NUM_9, SW12 PLUS_MINUS, SW13 DELETE, SW14 ENTER, SW15 SET_ZERO, SW16 SET_SPLN, SW17 ANG_ABS, SW18 ROT_CCW, SW19 RET_ZERO, SW2 NUM_4, SW20 NXT_SPLN, SW21 ANG_INC, SW22 ROT_CW, SW23 EXTRA_1, SW24 EXTRA_2, SW25 EXTRA_3, SW26 EXTRA_4, SW27 MODE_SWITCH, SW28 MULT_SWITCH, SW29 BOOT, SW3 NUM_7, SW30 RESET, SW4 DECIMAL, SW5 NUM_2, SW6 NUM_5, SW7 NUM_8, SW8 NUM_0, SW9 NUM_3, U1 ESP32-WROOM-32, U10 SN74LVC1T45DBV, U11 MAX3485, U12 MAX3485, U13 MAX3485, U2 74HC237, U3 SN74LVC1T45DBV, U4 SN74LVC1T45DBV, U5 XL1509-5.0, U6 XL1509-3.3, U7 SN74LVC1T45DBV, U8 SN74LVC1T45DBV, U9 SN74LVC1T45DBV

Commit message: please work
Other:
- board text added: "ENCB-"
Changed lines of the file:
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@@
-		)
-	)
-	(gr_text "GND"
-		(at 162.814 45.212 90)
-		(layer "B.SilkS")
-		(effects
-			(font
-				(size 1 1)
-				(thickness 0.15)
-			)
-			(justify left mirror)
 		)
 	)
 	(gr_text "ENCZ-"
-		(at 165.354 45.339 90)
+		(at 162.814 45.339 90)
 		(layer "B.SilkS")
 		(effects
@@
 	)
 	(gr_text "ENCZ+"
+		(at 165.354 45.212 90)
+		(layer "B.SilkS")
+		(effects
+			(font
+				(size 1 1)
+				(thickness 0.15)
+			)
+			(justify left mirror)
+		)
+	)
+	(gr_text "ENCB-"
 		(at 167.894 45.212 90)
 		(layer "B.SilkS")
