File: FourthAxis/KeyPad.kicad_sch (KiCad schematic)
At the start: 63 parts, among them SW1 NUM_1, SW10 NUM_6, SW11 NUM_9, SW12 PLUS_MINUS, SW13 DELETE, SW14 ENTER, SW15 SET_ZERO, SW16 SET_SPLN, SW17 ANG_ABS, SW18 ROT_CCW, SW19 RET_ZERO, SW2 NUM_4, SW20 NXT_SPLN, SW21 ANG_INC, SW22 ROT_CW, SW23 EXTRA_1, SW24 EXTRA_2, SW25 EXTRA_3, SW26 EXTRA_4, SW3 NUM_7, SW4 DECIMAL, SW5 NUM_2, SW6 NUM_5, SW7 NUM_8, SW8 NUM_0, SW9 NUM_3, U2 74HC237

Commit message: BOM export
Parts:
- SW1, SW10, SW11, SW12, SW13, SW14, SW15, SW16, SW17, SW18, SW19, SW2, SW20, SW21, SW22, SW23, SW24, SW25, SW26, SW3, SW4, SW5, SW6, SW7, SW8, SW9: now left out of the parts list
Changed lines of the file:
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@@
 		(body_style 1)
 		(exclude_from_sim no)
-		(in_bom yes)
+		(in_bom no)
 		(on_board yes)
 		(in_pos_files yes)
@@
 		(body_style 1)
 		(exclude_from_sim no)
-		(in_bom yes)
+		(in_bom no)
 		(on_board yes)
 		(in_pos_files yes)
@@
 		(body_style 1)
 		(exclude_from_sim no)
-		(in_bom yes)
+		(in_bom no)
 		(on_board yes)
 		(in_pos_files yes)
@@
 		(body_style 1)
 		(exclude_from_sim no)
-		(in_bom yes)
+		(in_bom no)
 		(on_board yes)
 		(in_pos_files yes)
@@
 		(body_style 1)
 		(exclude_from_sim no)
-		(in_bom yes)
+		(in_bom no)
 		(on_board yes)
 		(in_pos_files yes)
@@
 		(body_style 1)
 		(exclude_from_sim no)
-		(in_bom yes)
+		(in_bom no)
 		(on_board yes)
 		(in_pos_files yes)
@@
 		(body_style 1)
 		(exclude_from_sim no)
-		(in_bom yes)
+		(in_bom no)
 		(on_board yes)
 		(in_pos_files yes)
@@
 		(body_style 1)
 		(exclude_from_sim no)
-		(in_bom yes)
+		(in_bom no)
 		(on_board yes)
 		(in_pos_files yes)
@@
 		(body_style 1)
 		(exclude_from_sim no)
-		(in_bom yes)
+		(in_bom no)
 		(on_board yes)
 		(in_pos_files yes)
@@
 		(body_style 1)
 		(exclude_from_sim no)
-		(in_bom yes)
+		(in_bom no)
 		(on_board yes)
 		(in_pos_files yes)
@@
 		(body_style 1)
 		(exclude_from_sim no)
-		(in_bom yes)
+		(in_bom no)
 		(on_board yes)
 		(in_pos_files yes)
@@
 		(body_style 1)
 		(exclude_from_sim no)
-		(in_bom yes)
+		(in_bom no)
 		(on_board yes)
 		(in_pos_files yes)
@@
 		(body_style 1)
 		(exclude_from_sim no)
-		(in_bom yes)
+		(in_bom no)
 		(on_board yes)
 		(in_pos_files yes)
@@
 		(body_style 1)
 		(exclude_from_sim no)
-		(in_bom yes)
+		(in_bom no)
 		(on_board yes)
 		(in_pos_files yes)
@@
 		(body_style 1)
 		(exclude_from_sim no)
-		(in_bom yes)
+		(in_bom no)
 		(on_board yes)
 		(in_pos_files yes)
@@
 		(body_style 1)
 		(exclude_from_sim no)
-		(in_bom yes)
+		(in_bom no)
 		(on_board yes)
 		(in_pos_files yes)
@@
 		(body_style 1)
 		(exclude_from_sim no)
-		(in_bom yes)
+		(in_bom no)
 		(on_board yes)
 		(in_pos_files yes)
@@
 		(body_style 1)
 		(exclude_from_sim no)
-		(in_bom yes)
+		(in_bom no)
 		(on_board yes)
 		(in_pos_files yes)
@@
 		(body_style 1)
 		(exclude_from_sim no)
-		(in_bom yes)
+		(in_bom no)
 		(on_board yes)
 		(in_pos_files yes)
@@
 		(body_style 1)
 		(exclude_from_sim no)
-		(in_bom yes)
+		(in_bom no)
 		(on_board yes)
 		(in_pos_files yes)
@@
 		(body_style 1)
 		(exclude_from_sim no)
-		(in_bom yes)
+		(in_bom no)
 		(on_board yes)
 		(in_pos_files yes)
@@
 		(body_style 1)
 		(exclude_from_sim no)
-		(in_bom yes)
+		(in_bom no)
 		(on_board yes)
 		(in_pos_files yes)
@@
 		(body_style 1)
 		(exclude_from_sim no)
-		(in_bom yes)
+		(in_bom no)
 		(on_board yes)
 		(in_pos_files yes)
@@
 		(body_style 1)
 		(exclude_from_sim no)
-		(in_bom yes)
+		(in_bom no)
 		(on_board yes)
 		(in_pos_files yes)
@@
 		(body_style 1)
 		(exclude_from_sim no)
-		(in_bom yes)
+		(in_bom no)
 		(on_board yes)
 		(in_pos_files yes)
@@
 		(body_style 1)
 		(exclude_from_sim no)
-		(in_bom yes)
+		(in_bom no)
 		(on_board yes)
 		(in_pos_files yes)

Commit message: boards ordered
Parts:
- D1, D10, D11, D12, D13, D14, D15, D16, D17, D18, D19, D2, D20, D21, D22, D23, D24, D25, D26, D3, D4, D5, D6, D7, D8, D9: value D -> 1N5821
Changed lines of the file:
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@@
 			)
 		)
-		(property "Value" "D"
+		(property "Value" "1N5821"
 			(at 129.54 118.11 0)
 			(show_name no)
@@
 			)
 		)
-		(property "Value" "D"
+		(property "Value" "1N5821"
 			(at 172.72 118.11 0)
 			(show_name no)
@@
 			)
 		)
-		(property "Value" "D"
+		(property "Value" "1N5821"
 			(at 107.95 104.14 0)
 			(show_name no)
@@
 			)
 		)
-		(property "Value" "D"
+		(property "Value" "1N5821"
 			(at 215.9 76.2 0)
 			(show_name no)
@@
 			)
 		)
-		(property "Value" "D"
+		(property "Value" "1N5821"
 			(at 151.13 104.14 0)
 			(show_name no)
@@
 			)
 		)
-		(property "Value" "D"
+		(property "Value" "1N5821"
 			(at 237.49 76.2 0)
 			(show_name no)
@@
 			)
 		)
-		(property "Value" "D"
+		(property "Value" "1N5821"
 			(at 194.31 76.2 0)
 			(show_name no)
@@
 			)
 		)
-		(property "Value" "D"
+		(property "Value" "1N5821"
 			(at 237.49 90.17 0)
 			(show_name no)
@@
 			)
 		)
-		(property "Value" "D"
+		(property "Value" "1N5821"
 			(at 151.13 118.11 0)
 			(show_name no)
@@
 			)
 		)
-		(property "Value" "D"
+		(property "Value" "1N5821"
 			(at 215.9 90.17 0)
 			(show_name no)
@@
 			)
 		)
-		(property "Value" "D"
+		(property "Value" "1N5821"
 			(at 237.49 104.14 0)
 			(show_name no)
@@
 			)
 		)
-		(property "Value" "D"
+		(property "Value" "1N5821"
 			(at 215.9 118.11 0)
 			(show_name no)
@@
 			)
 		)
-		(property "Value" "D"
+		(property "Value" "1N5821"
 			(at 129.54 104.14 0)
 			(show_name no)
@@
 			)
 		)
-		(property "Value" "D"
+		(property "Value" "1N5821"
 			(at 151.13 90.17 0)
 			(show_name no)
@@
 			)
 		)
-		(property "Value" "D"
+		(property "Value" "1N5821"
 			(at 172.72 104.14 0)
 			(show_name no)
@@
 			)
 		)
-		(property "Value" "D"
+		(property "Value" "1N5821"
 			(at 237.49 118.11 0)
 			(show_name no)
@@
 			)
 		)
-		(property "Value" "D"
+		(property "Value" "1N5821"
 			(at 107.95 90.17 0)
 			(show_name no)
@@
 			)
 		)
-		(property "Value" "D"
+		(property "Value" "1N5821"
 			(at 215.9 104.14 0)
 			(show_name no)
@@
 			)
 		)
-		(property "Value" "D"
+		(property "Value" "1N5821"
 			(at 151.13 76.2 0)
 			(show_name no)
@@
 			)
 		)
-		(property "Value" "D"
+		(property "Value" "1N5821"
 			(at 194.31 90.17 0)
 			(show_name no)
@@
 			)
 		)
-		(property "Value" "D"
+		(property "Value" "1N5821"
 			(at 194.31 104.14 0)
 			(show_name no)
@@
 			)
 		)
-		(property "Value" "D"
+		(property "Value" "1N5821"
 			(at 129.54 76.2 0)
 			(show_name no)
@@
 			)
 		)
-		(property "Value" "D"
+		(property "Value" "1N5821"
 			(at 107.95 118.11 0)
 			(show_name no)
@@
 			)
 		)
-		(property "Value" "D"
+		(property "Value" "1N5821"
 			(at 107.95 76.2 0)
 			(show_name no)
@@
 			)
 		)
-		(property "Value" "D"
+		(property "Value" "1N5821"
 			(at 194.31 118.11 0)
 			(show_name no)
@@
 			)
 		)
-		(property "Value" "D"
+		(property "Value" "1N5821"
 			(at 129.54 90.17 0)
 			(show_name no)
